Commit message: made the rbvogui_plus ignition-compatible; added onRobot RG6 gripper to rbvogui_plus

File: robots/rbvogui/rbvogui_plus.urdf.xacro (robot description, xacro)
@@ -18,8 +18,11 @@
   <xacro:arg
     name="gazebo_ignition"
-    default="false" />
+    default="true" />
   <xacro:arg
     name="ur_type"
     default="ur5e" />
+  <xacro:arg
+    name="end_effector"
+    default="rg6" />
   <!-- RB-VOGUI -->
   <xacro:rbvogui
@@ -32,5 +35,6 @@
     frame_prefix="$(arg prefix)arm_"
     parent="$(arg prefix)chassis_link"
-    gazebo_ignition="$(arg gazebo_ignition)">
+    gazebo_ignition="$(arg gazebo_ignition)"
+    end_effector="$(arg end_effector)">
     <origin
       xyz="0 0 0.235"
@@ -53,7 +57,7 @@
     node_namespace="$(arg namespace)"
     node_name="front_laser"
-    gazebo_ignition="$(arg gazebo_ignition)"
-    max_angle="2.1"
-    min_angle="-2.1">
+    gazebo_ignition="$(arg gazebo_ignition)">
+    <!-- max_angle="2.1"
+    min_angle="-2.1" -->
     <origin
       xyz="0.53 0.33 0.1145"
@@ -65,7 +69,7 @@
     node_namespace="$(arg namespace)"
     node_name="rear_laser"
-    gazebo_ignition="$(arg gazebo_ignition)"
-    max_angle="2.1"
-    min_angle="-2.1">
+    gazebo_ignition="$(arg gazebo_ignition)">
+    <!-- max_angle="2.1"
+    min_angle="-2.1" -->
     <origin
       xyz="-0.53 -0.33 0.1145"

File: urdf/arms/ur_macro.urdf.xacro (robot description, xacro)
@@ -6,4 +6,6 @@
   <xacro:include
     filename="$(find ur_description)/urdf/ur_macro.xacro" />
+  <xacro:include filename="$(find campetella_sim)/models/2f_85/urdf/robotiq_2f_85_macro.urdf.xacro" />
+  <xacro:include filename="$(find campetella_sim)/models/sd_35/urdf/sd_25_macro.urdf.xacro" />
   <xacro:macro
     name="arm_ur"
@@ -13,5 +15,6 @@
     *origin
     parent
-    gazebo_ignition:=false
+    gazebo_ignition:=true
+    end_effector:='none'
     ">
     <xacro:property
@@ -34,20 +37,44 @@
       kinematics_parameters_file="${kinematics_params}"
       physical_parameters_file="${physical_params}"
-      visual_parameters_file="${visual_params}"
-      generate_ros2_control_tag="false">
+      visual_parameters_file="${visual_params}">
       <xacro:insert_block name="origin" />
     </xacro:ur_robot>
+    <!-- Onrobot RG6 -->
+    <xacro:if value="${end_effector == 'rg6'}">
+      <xacro:include filename="$(find onrobot_rg_description)/urdf/onrobot_rg6_model_macro.xacro" />
+      <xacro:onrobot_rg6 prefix="${frame_prefix}rg6_" gazebo_ignition="${gazebo_ignition}"/>
+      <joint name="${frame_prefix}joint_tcp_fixed" type="fixed">
+          <parent link="${frame_prefix}tool0"/>
+          <child link="${frame_prefix}rg6_base_link"/>
+          <origin rpy="0 0 0" xyz="0 0.0 0.0"/>
+      </joint>
+    </xacro:if>
+    <!-- Robotiq 2F-85 -->
+    <xacro:if value="${end_effector == '2f85'}">
+      <xacro:robotiq_gripper
+            name="robotiq_2f_85"
+            prefix="${frame_prefix}gripper_"
+            parent="${frame_prefix}tool0"
+            sim_ignition="true"
+            include_ros2_control="true">
+            <origin xyz="0.0 0 0" rpy="0 0 0"/>
+        </xacro:robotiq_gripper>
+    </xacro:if>
+    <!-- Screwdriver -->
+    <xacro:if value="${end_effector == 'screwdriver'}">
+        <xacro:sd_25_screwdrivew
+            scale="0.001"
+            parent="${frame_prefix}tool0"
+            xyz="0 0.095 0.065"
+            rpy="3.14 0 0"
+        />
+    </xacro:if>
     <xacro:if value="$(arg gazebo_ignition)">
       <xacro:include
-        filename="$(find ur_description)/urdf/ur.ros2_control.xacro" />
+        filename="$(find ur_simulation_gz)/urdf/ur_gz.ros2_control.xacro" />
       <xacro:ur_ros2_control
         name="arm"
-        sim_ignition="true"
         tf_prefix="${frame_prefix}"
-        script_filename=""
-        output_recipe_filename=""
-        input_recipe_filename=""
-        hash_kinematics=""
-        robot_ip="" />
+         />
     </xacro:if>
   </xacro:macro>

Commit message: added tool changing parts on the rbvogui_plus urdf

File: robots/rbvogui/rbvogui_plus.urdf.xacro (robot description, xacro)
@@ -9,4 +9,5 @@
   <xacro:include
     filename="$(find robotnik_sensors)/urdf/all_sensors.urdf.xacro" />
+  <xacro:include filename="$(find campetella_sim)/models/tool_changer/urdf/tool_changer_macro.urdf.xacro" />
   <!-- ARGUMENTS -->
   <xacro:arg
@@ -30,4 +31,11 @@
     gazebo_ignition="$(arg gazebo_ignition)"
     namespace="$(arg namespace)" />
+  <!-- TOOL CHANGER -->
+  <xacro:tool_changer
+        parent="$(arg prefix)base_link"
+        prefix="$(arg prefix)tc_"
+        xyz="0.0 0.0 0.402"
+        rpy="0 0 1.57"
+    />
   <!-- ARMS -->
   <xacro:arm_ur
@@ -37,6 +45,7 @@
     gazebo_ignition="$(arg gazebo_ignition)"
     end_effector="$(arg end_effector)">
+    <!-- Correct the origin of the arm below: -->
     <origin
-      xyz="0 0 0.235"
+      xyz="0.08 0.0 0.25"
       rpy="0 0 0" />
   </xacro:arm_ur>

File: urdf/arms/ur_macro.urdf.xacro (robot description, xacro)
@@ -6,6 +6,7 @@
   <xacro:include
     filename="$(find ur_description)/urdf/ur_macro.xacro" />
-  <xacro:include filename="$(find campetella_sim)/models/2f_85/urdf/robotiq_2f_85_macro.urdf.xacro" />
-  <xacro:include filename="$(find campetella_sim)/models/sd_35/urdf/sd_25_macro.urdf.xacro" />
+  <!-- <xacro:include filename="$(find campetella_sim)/models/2f_85/urdf/robotiq_2f_85_macro.urdf.xacro" /> -->
+  <!-- <xacro:include filename="$(find campetella_sim)/models/sd_35/urdf/sd_25_macro.urdf.xacro" /> -->
+  <xacro:property name="initial_positions" value="${xacro.load_yaml('$(find ur_description)/config/initial_positions.yaml')}"/>
   <xacro:macro
     name="arm_ur"
@@ -76,5 +77,5 @@
         name="arm"
         tf_prefix="${frame_prefix}"
-         />
+        initial_positions="${initial_positions}" />
     </xacro:if>
   </xacro:macro>
