Commit message: add ur camera to rbvogui_plus

File: robots/rbvogui/rbvogui_plus.urdf.xacro (robot description, xacro)
@@ -11,4 +11,5 @@
   <xacro:include filename="$(find campetella_sim)/models/tool_changer/urdf/tool_changer_macro.urdf.xacro" />
   <xacro:include filename="$(find campetella_sim)/models/tool_changer/urdf/tool_changer_detachable_joints.urdf.xacro" />
+  <xacro:include filename="$(find campetella_sim)/models/ur_wrist_camera/urdf/ur_wrist_camera.urdf.xacro" />
   <!-- ARGUMENTS -->
   <xacro:arg
@@ -112,4 +113,13 @@
       rpy="0 0 -${pi}" />
   </xacro:sensor_intel_realsense_d435>
+  <!-- WRIST CAMERA-->
+  <xacro:ur_wrist_camera
+    prefix="$(arg prefix)arm_rgbd_camera_"
+    parent="$(arg prefix)arm_tool0"
+    node_namespace="$(arg namespace)"
+    node_name="arm_camera"
+    gazebo_ignition="$(arg gazebo_ignition)">
+    <origin xyz="0 0 0" rpy="0 0 0" />
+  </xacro:ur_wrist_camera>
   <!-- DETACHABLE TOOL JOINTS (4 tools × 2 joints = 8 DetachableJoint plugins) -->
   <xacro:if value="$(arg use_tool_changer)">

Commit message: update position of camera adapter with tool changing component

File: robots/rbvogui/rbvogui_plus.urdf.xacro (robot description, xacro)
@@ -11,5 +11,4 @@
   <xacro:include filename="$(find campetella_sim)/models/tool_changer/urdf/tool_changer_macro.urdf.xacro" />
   <xacro:include filename="$(find campetella_sim)/models/tool_changer/urdf/tool_changer_detachable_joints.urdf.xacro" />
-  <xacro:include filename="$(find campetella_sim)/models/ur_wrist_camera/urdf/ur_wrist_camera.urdf.xacro" />
   <!-- ARGUMENTS -->
   <xacro:arg
@@ -49,5 +48,7 @@
     parent="$(arg prefix)chassis_link"
     gazebo_ignition="$(arg gazebo_ignition)"
-    end_effector="$(arg end_effector)">
+    end_effector="$(arg end_effector)"
+    has_wrist_camera="true"
+    node_namespace="$(arg namespace)">
     <!-- Correct the origin of the arm below: -->
     <origin
@@ -111,13 +112,4 @@
       rpy="0 0 -${pi}" />
   </xacro:sensor_intel_realsense_d435>
-  <!-- WRIST CAMERA-->
-  <xacro:ur_wrist_camera
-    prefix="$(arg prefix)arm_rgbd_camera_"
-    parent="$(arg prefix)arm_tool0"
-    node_namespace="$(arg namespace)"
-    node_name="arm_camera"
-    gazebo_ignition="$(arg gazebo_ignition)">
-    <origin xyz="0 0 0" rpy="0 0 0" />
-  </xacro:ur_wrist_camera>
   <!-- DETACHABLE TOOL JOINTS (4 tools × 2 joints = 8 DetachableJoint plugins) -->
   <xacro:if value="$(arg use_tool_changer)">

File: urdf/arms/ur_macro.urdf.xacro (robot description, xacro)
@@ -8,4 +8,6 @@
   <!-- <xacro:include filename="$(find campetella_sim)/models/2f_85/urdf/robotiq_2f_85_macro.urdf.xacro" /> -->
   <!-- <xacro:include filename="$(find campetella_sim)/models/sd_35/urdf/sd_35_macro.urdf.xacro" /> -->
+  <xacro:include
+    filename="$(find campetella_sim)/models/ur_wrist_camera/urdf/ur_wrist_camera.urdf.xacro" />
   <xacro:property name="initial_positions" value="${xacro.load_yaml('initial_positions.yaml')}"/>
   <xacro:macro
@@ -18,4 +20,6 @@
     gazebo_ignition:=true
     end_effector:='none'
+    has_wrist_camera:=false
+    node_namespace:=''
     ">
     <xacro:property
@@ -71,4 +75,41 @@
         />
     </xacro:if>
+    <!-- Wrist camera: flange -> camera adapter -> tool changer robot side -->
+    <xacro:if value="${has_wrist_camera}">
+      <xacro:ur_wrist_camera
+        prefix="${frame_prefix}rgbd_camera_"
+        parent="${frame_prefix}flange"
+        node_namespace="${node_namespace}"
+        node_name="arm_camera"
+        gazebo_ignition="${gazebo_ignition}">
+        <origin xyz="0 0 0" rpy="${pi/2.0} 0 ${pi/2.0}" />
+      </xacro:ur_wrist_camera>
+      <!-- Tool Changer Robot Side: permanently attached to the camera adapter; used as planning target when no tool is attached -->
+      <link name="${frame_prefix}tc_robot_side">
+        <inertial>
+          <mass value="0.3"/>
+          <origin xyz="0 0 0" rpy="0 0 0"/>
+          <inertia ixx="0.0005" ixy="0" ixz="0" iyy="0.0005" iyz="0" izz="0.0005"/>
+        </inertial>
+        <visual>
+          <geometry>
+            <mesh filename="file://$(find campetella_sim)/models/tool_changer/meshes/tc_robot_side.stl" scale="0.001 0.001 0.001"/>
+          </geometry>
+          <material name="silver">
+            <color rgba="0.75 0.75 0.75 1.0"/>
+          </material>
+        </visual>
+        <collision>
+          <geometry>
+            <mesh filename="file://$(find campetella_sim)/models/tool_changer/meshes/tc_robot_side.stl" scale="0.001 0.001 0.001"/>
+          </geometry>
+        </collision>
+      </link>
+      <joint name="${frame_prefix}tc_robot_side_joint" type="fixed">
+        <parent link="${frame_prefix}rgbd_camera_bracket_link"/>
+        <child link="${frame_prefix}tc_robot_side"/>
+        <origin xyz="0.0 0.0 0.0" rpy="0 0 0"/>
+      </joint>
+    </xacro:if>
     <xacro:if value="$(arg gazebo_ignition)">
       <xacro:include

Commit message: update description for real hardware

File: robots/rbvogui/rbvogui_plus.urdf.xacro (robot description, xacro)
@@ -30,4 +30,12 @@
     name="use_tool_changer"
     default="true" />
+  <!-- Optional model parameters supplied by ur_robot_driver on real hardware. -->
+  <xacro:arg name="joint_limit_params" default="" />
+  <xacro:arg name="kinematics_params" default="" />
+  <xacro:arg name="physical_params" default="" />
+  <xacro:arg name="visual_params" default="" />
+  <xacro:arg name="safety_limits" default="false" />
+  <xacro:arg name="safety_pos_margin" default="0.15" />
+  <xacro:arg name="safety_k_position" default="20" />
   <xacro:arg
     name="wrist_camera"
@@ -54,5 +62,12 @@
     has_wrist_camera="true"
     node_namespace="$(arg namespace)"
-    wrist_camera="$(arg wrist_camera)">
+    wrist_camera="$(arg wrist_camera)"
+    joint_limit_params_file="$(arg joint_limit_params)"
+    kinematics_params_file="$(arg kinematics_params)"
+    physical_params_file="$(arg physical_params)"
+    visual_params_file="$(arg visual_params)"
+    safety_limits="$(arg safety_limits)"
+    safety_pos_margin="$(arg safety_pos_margin)"
+    safety_k_position="$(arg safety_k_position)">
     <!-- Correct the origin of the arm below: -->
     <origin

File: urdf/arms/ur_macro.urdf.xacro (robot description, xacro)
@@ -23,17 +23,30 @@
     node_namespace:=''
     wrist_camera:='stereolabs_zed2i'
+    joint_limit_params_file:=''
+    kinematics_params_file:=''
+    physical_params_file:=''
+    visual_params_file:=''
+    safety_limits:=false
+    safety_pos_margin:=0.15
+    safety_k_position:=20
     ">
-    <xacro:property
-      name="joint_limit_params"
-      default="$(find ur_description)/config/$(arg ur_type)/joint_limits.yaml" />
-    <xacro:property
-      name="kinematics_params"
-      default="$(find ur_description)/config/$(arg ur_type)/default_kinematics.yaml" />
-    <xacro:property
-      name="physical_params"
-      default="$(find ur_description)/config/$(arg ur_type)/physical_parameters.yaml" />
-    <xacro:property
-      name="visual_params"
-      default="$(find ur_description)/config/$(arg ur_type)/visual_parameters.yaml" />
+    <xacro:property name="default_joint_limit_params"
+      value="$(find ur_description)/config/$(arg ur_type)/joint_limits.yaml" />
+    <xacro:property name="default_kinematics_params"
+      value="$(find ur_description)/config/$(arg ur_type)/default_kinematics.yaml" />
+    <xacro:property name="default_physical_params"
+      value="$(find ur_description)/config/$(arg ur_type)/physical_parameters.yaml" />
+    <xacro:property name="default_visual_params"
+      value="$(find ur_description)/config/$(arg ur_type)/visual_parameters.yaml" />
+    <!-- A non-empty real-hardware argument wins; simulation keeps the
+         description package defaults. -->
+    <xacro:property name="joint_limit_params"
+      value="${joint_limit_params_file or default_joint_limit_params}" />
+    <xacro:property name="kinematics_params"
+      value="${kinematics_params_file or default_kinematics_params}" />
+    <xacro:property name="physical_params"
+      value="${physical_params_file or default_physical_params}" />
+    <xacro:property name="visual_params"
+      value="${visual_params_file or default_visual_params}" />
     <xacro:ur_robot
       name="${ur_type}"
@@ -44,4 +57,7 @@
       physical_parameters_file="${physical_params}"
       visual_parameters_file="${visual_params}"
+      safety_limits="${safety_limits}"
+      safety_pos_margin="${safety_pos_margin}"
+      safety_k_position="${safety_k_position}"
     >
       <xacro:insert_block name="origin" />
@@ -78,5 +94,8 @@
     </xacro:if>
     <!-- Wrist camera: flange -> camera adapter -> tool changer robot side -->
-    <xacro:if value="${has_wrist_camera}">
+    <!-- `wrist_camera:=none` intentionally expands the camera macro to no
+         links.  Gate the complete camera/tool-changer branch as well, or the
+         tool-changer joint would reference a non-existent bracket link. -->
+    <xacro:if value="${has_wrist_camera and wrist_camera != 'none'}">
       <xacro:ur_wrist_camera
         prefix="${frame_prefix}rgbd_camera_"
